File: organ switches v1.kicad_pcb (KiCad board)
At the start: 2 copper layers, 76.2 x 76.2 mm, 74 parts, among them J1 Conn_01x08, J2 Conn_01x08, SW1 SW_SPST, SW10 SW_SPST, SW11 SW_SPST, SW12 SW_SPST, SW13 SW_SPST, SW14 SW_SPST, SW15 SW_SPST, SW16 SW_SPST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

Commit message: Add files via upload
Parts:
- removed ? (x4): MountingHole_2.2mm_M2, MountingHole:MountingHole_2.2mm_M2
- added C1: 0.1uF, Capacitor_SMD:C_0603_1608Metric_Pad1.05x0.95mm_HandSolder, B.Cu at (228.6, 87.5)
- added C2: 0.1uF, Capacitor_SMD:C_0603_1608Metric_Pad1.05x0.95mm_HandSolder, B.Cu at (215.3, 124.5)
- added C3: 0.1uF, Capacitor_SMD:C_0603_1608Metric_Pad1.05x0.95mm_HandSolder, B.Cu at (266.2, 86.3)
- added C4: 0.1uF, Capacitor_SMD:C_0603_1608Metric_Pad1.05x0.95mm_HandSolder, B.Cu at (265.9, 123.3)
- added H1: MountingHole, MountingHole:MountingHole_3mm, F.Cu at (211.5, 89.4)
- added H2: MountingHole, MountingHole:MountingHole_3mm, F.Cu at (205.2, 142.7)
- added H3: MountingHole, MountingHole:MountingHole_3mm, F.Cu at (269.7, 88.9)
- added H4: MountingHole, MountingHole:MountingHole_3mm, F.Cu at (274.9, 142.8)
- added J3: Conn_01x04, Connector_PinHeader_2.54mm:PinHeader_1x04_P2.54mm_Vertical, F.Cu at (277.1, 82.7)
- added J4: Conn_01x04, Connector_PinHeader_2.54mm:PinHeader_1x04_P2.54mm_Vertical, F.Cu at (277.1, 120.6)
- D1, D10, D11, D12, D13, D14, D15, D16, D2, D3, D4, D5, D6, D7, D8, D9: footprint LED_THT:LED_D3.0mm -> LED_THT:LED_D3.0mm_with_sockets
- J1, J2: value Conn_01x08 -> Conn_01x04; footprint Connector_PinHeader_2.54mm:PinHeader_1x08_P2.54mm_Vertical -> Connector_PinHeader_2.54mm:PinHeader_1x04_P2.54mm_Vertical; moved to F.Cu
- U3, U4: value TLC6C598QPWRQ1 -> TLC6C598CQDRQ1; footprint eec:Texas_Instruments-PW0016A-0-0-0 -> Package_SO:SOIC-16_3.9x9.9mm_P1.27mm
- moved J1 77.1 mm to (203.0, 82.7), turned to 0 degrees
- moved U3 26.8 mm to (259.9, 86.0), turned to 270 degrees
- moved U1 20.7 mm to (221.9, 85.8), turned to 90 degrees
- moved U4 18.9 mm to (259.8, 124.2)
- moved R17 14.1 mm to (274.3, 72.0), turned to 0 degrees
- moved R32 12.9 mm to (219.2, 135.4), turned to 90 degrees
- moved J2 12.1 mm to (203.0, 120.7), turned to 0 degrees
- moved R25 11.9 mm to (274.9, 110.0), turned to 180 degrees
- moved R31 10.9 mm to (237.3, 129.1)
- moved R21 10.8 mm to (275.9, 97.3), turned to 90 degrees
- moved R24 10.7 mm to (219.1, 97.2), turned to 90 degrees
- moved R23 9.48 mm to (237.2, 90.8)
- moved R3 9.10 mm to (234.8, 83.3), turned to 90 degrees
- moved R1 8.48 mm to (273.0, 83.7), turned to 90 degrees
- moved R9 8.38 mm to (272.0, 125.5), turned to 180 degrees
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Connections:
- net Net-(J1-Pad4) renamed /SW_DOUT
- J1 pad 2: Net-(J1-Pad2) -> /SW_CLK
- J1 pad 3: Net-(J1-Pad3) -> /SW_LOAD
- J2 pad 1: +5V -> /LED_DIN
- J2 pad 2: Net-(J1-Pad2) -> /LED_LOAD
- J2 pad 3: Net-(J1-Pad3) -> /LED_CLK
- J2 pad 4: Net-(J2-Pad4) -> GND
- U1 pad 1: Net-(J1-Pad3) -> /SW_LOAD
- U1 pad 2: Net-(J1-Pad2) -> /SW_CLK
- U2 pad 1: Net-(J1-Pad3) -> /SW_LOAD
- U2 pad 10: Net-(J2-Pad4) -> /SW_DIN
- U2 pad 16: Net-(U2-Pad16) -> +5V
- U2 pad 2: Net-(J1-Pad2) -> /SW_CLK
- U3 pad 10: Net-(J1-Pad6) -> /LED_LOAD
- U3 pad 15: Net-(J1-Pad7) -> /LED_CLK
- U3 pad 2: Net-(J1-Pad5) -> /LED_DIN
- U4 pad 10: Net-(J1-Pad6) -> /LED_LOAD
- U4 pad 15: Net-(J1-Pad7) -> /LED_CLK
- U4 pad 9: Net-(J2-Pad5) -> /LED_DOUT
Routing:
- net /SW_CLK: track 0.00 -> 194.6 mm, vias 0 -> 9
- net Net-(J1-Pad3): track 186.1 -> 0.00 mm, vias 3 -> 0
- net Net-(J1-Pad2): track 173.3 -> 0.00 mm, vias 6 -> 0
- net /LED_LOAD: track 0.00 -> 171.8 mm, vias 0 -> 9
- net /SW_LOAD: track 0.00 -> 158.5 mm, vias 0 -> 9
- net /LED_CLK: track 0.00 -> 150.3 mm, vias 0 -> 7
- net /SW_DIN: track 0.00 -> 119.3 mm, vias 0 -> 4
- net GND: track 154.4 -> 50.7 mm, vias 23 -> 27
- net /LED_DIN: track 0.00 -> 96.3 mm, vias 0 -> 5
- net Net-(J1-Pad6): track 75.7 -> 0.00 mm, vias 2 -> 0
- net Net-(J1-Pad7): track 65.3 -> 0.00 mm, vias 1 -> 0
- net +5V: track 55.8 -> 0.00 mm, vias 10 -> 0
- net Net-(R20-Pad2): track 75.0 -> 22.7 mm
- net Net-(J2-Pad5): track 38.9 -> 0.00 mm, vias 3 -> 0
- net Net-(D8-Pad1): track 29.5 -> 64.0 mm, vias 0 -> 1
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Other:
- board size 76.2 x 76.2 mm -> 76.2 x 76.3 mm
